Commit message: Update codes after last changes

File: src/mobile_manipulator_sim/urdf/simple_mobile_robot.urdf (robot description, URDF)
Before this commit: robot simple_mobile_robot, 13 links, 12 joints
Links:
- added link camera_link, mass 0.1; collision box size=0.03 0.08 0.03; visual box size=0.03 0.08 0.03
Joints:
- added joint camera_joint: type fixed, parent base_link, child camera_link, origin xyz=0 0 0.05 rpy=0 1.5708 0

Commit message: IMU Added Successfuly !

File: src/mobile_manipulator_sim/urdf/simple_mobile_robot.urdf (robot description, URDF)
Before this commit: robot simple_mobile_robot, 14 links, 13 joints
Links:
- added link imu_link, mass 0.01; collision box size=0.05 0.05 0.02; visual box size=0.05 0.05 0.02
Joints:
- added joint imu_joint: type fixed, parent base_link, child imu_link, origin xyz=0 0 0.05 rpy=0 0 0
